File: LibreScale_HW/LibreScale_HW.kicad_sch (KiCad schematic)
At the start: 15 parts

Commit message: Minor changes
Parts:
- added J?: AVR-UPDI-6, Connector:Tag-Connect_TC2030-IDC-NL_2x03_P1.27mm_Vertical, symbol Connector:AVR-UPDI-6
- C3: renamed from C?; footprint (none) -> Capacitor_SMD:C_0603_1608Metric
- JP1: footprint (none) -> Jumper:SolderJumper-2_P1.3mm_Bridged_RoundedPad1.0x1.5mm
- R3: renamed from R?; footprint (none) -> Resistor_SMD:R_0402_1005Metric_Pad0.72x0.64mm_HandSolder
- R4: renamed from R?; value R_Small -> 1k; footprint (none) -> Resistor_SMD:R_0402_1005Metric_Pad0.72x0.64mm_HandSolder
- R_{G}1: renamed from R_{G}; footprint (none) -> Resistor_SMD:R_0402_1005Metric_Pad0.72x0.64mm_HandSolder
- U2: renamed from U?; footprint (none) -> Package_SO:SOIC-8_3.9x4.9mm_P1.27mm
- gave numbers to parts that had none: 4
- renumbered R_{strain} to R_{strain}1, R_{strain} to R_{strain}2
Connections:
- net V_{meas+} is gone; now on net V_{meas}+: U3.3 (+)
- net V_{meas-} is gone; now on net V_{meas}-: U3.2 (-)
- net +5V: now also J?.2 (VCC)
- net GND: now also J?.6 (GND)
- net UDPI: now also J?.1 (DATA)
- net V_{out}: now also R4.2; no longer C3.1, U2.2 (IN+)
- net at R4.1: now also C3.1, U2.2 (IN+)
Other:
- note added: "Analog-To-Digital-Converter"
- note added: "Input-amplifier OpAmp"
- note added: "MCU"
- note added: "Wheatstone bridge"
- moved on the sheet: C2, R4, U1

Commit message: minor fixes on PCB
Parts:
- added H1, H2, H5, H6: MountingHolePCB, MountingHole:MountingHole_3.2mm_M3_Pad, symbol Mechanical:MountingHole
- added H3, H4: MountingHoleLoad, MountingHole:MountingHole_3.2mm_M3_DIN965_Pad, symbol Mechanical:MountingHole
- R1, R2: value R -> 1k
- R_{strain}1, R_{strain}2: footprint Connector_PinHeader_2.54mm:PinHeader_1x02_P2.54mm_Vertical -> Connector_JST:JST_PH_S2B-PH-K_1x02_P2.00mm_Horizontal
- gave numbers to parts that had none: 1
Connections:
- net CLK is gone; now on net SCK: U2.7 (CLK)
- net D_{out} is gone; now on net MISO: U2.6 (Dout)
