File: LibreScale_HW/LibreScale_HW.kicad_pcb (KiCad board)
At the start: 2 copper layers, 15 parts, among them U1 ATtiny402-SS, U2 MCP3301, U3 INA333xxDGK

Commit message: minor fixes on PCB
Parts:
- added H1: MountingHolePCB, MountingHole:MountingHole_3.2mm_M3_Pad, F.Cu at (90.0, 110.0)
- added H2: MountingHolePCB, MountingHole:MountingHole_3.2mm_M3_Pad, F.Cu at (130.0, 166.0)
- added H3: MountingHoleLoad, MountingHole:MountingHole_3.2mm_M3_DIN965_Pad, F.Cu at (89.9, 143.0)
- added H5: MountingHolePCB, MountingHole:MountingHole_3.2mm_M3_Pad, F.Cu at (130.0, 110.0)
- added H6: MountingHolePCB, MountingHole:MountingHole_3.2mm_M3_Pad, F.Cu at (90.0, 166.0)
- added H7: MountingHoleLoad, MountingHole:MountingHole_3.2mm_M3_DIN965_Pad, F.Cu at (89.9, 137.0)
- added J1: AVR-UPDI-6, Connector:Tag-Connect_TC2030-IDC-NL_2x03_P1.27mm_Vertical, F.Cu at (107.3, 151.1)
- R1, R2: value R -> 1k
- R_{strain}1, R_{strain}2: footprint Connector_PinHeader_2.54mm:PinHeader_1x02_P2.54mm_Vertical -> Connector_JST:JST_PH_S2B-PH-K_1x02_P2.00mm_Horizontal
- moved R2 119.4 mm to (115.1, 162.0), turned to 180 degrees
- moved C1 108.4 mm to (108.6, 163.7), turned to 0 degrees
- moved D1 105.9 mm to (104.0, 164.3)
- moved R3 105.9 mm to (101.0, 163.7)
- moved U2 105.9 mm to (100.2, 159.8)
- moved U3 105.9 mm to (113.1, 159.4)
- moved C3 105.9 mm to (105.6, 159.1)
- moved R4 105.9 mm to (108.3, 159.1)
- moved R_{G}1 105.9 mm to (111.5, 162.1)
- moved R1 105.9 mm to (115.1, 163.8), turned to 0 degrees
- moved C2 104.8 mm to (98.0, 148.3)
- moved U1 104.8 mm to (100.2, 151.8)
- moved R_{strain}1 102.8 mm to (126.5, 160.0), turned to 90 degrees
- moved R_{strain}2 102.8 mm to (126.5, 151.2), turned to 90 degrees
- moved JP1 98.7 mm to (97.7, 155.8), turned to 180 degrees
Connections:
- U2 pad 6: /D_{out} -> /MISO
- U2 pad 7: /CLK -> /SCK
Routing:
- net +5V: track 20.8 -> 59.4 mm
- net /SCK: track 0.00 -> 16.6 mm
- net /MISO: track 0.00 -> 12.8 mm
- net GND: track 0.00 -> 10.9 mm, vias 0 -> 4
- net /V_{ref}: track 3.71 -> 13.9 mm, vias 0 -> 2
- net /UDPI: track 0.00 -> 10.1 mm
- net /V_{meas}+: track 17.3 -> 11.7 mm
- net /CS1: track 8.69 -> 12.3 mm
- net /V_{meas}-: track 8.50 -> 5.55 mm
Other:
- board outline added: 52 x 68 mm

Commit message: Routing changes, added parts
Parts:
- removed H3, H7: MountingHoleLoad, MountingHole:MountingHole_3.2mm_M3_DIN965_Pad
- added BT1: Battery_Cell, Connector_JST:JST_PH_S2B-PH-K_1x02_P2.00mm_Horizontal, F.Cu at (136.7, 100.3)
- moved R3 78.0 mm to (152.2, 104.8)
- moved C3 78.0 mm to (156.8, 100.2)
- moved D1 78.0 mm to (155.2, 105.4)
- moved R1 78.0 mm to (166.3, 104.9)
- moved R2 78.0 mm to (166.3, 103.1)
- moved R_{G}1 78.0 mm to (162.7, 103.2)
- moved U2 78.0 mm to (151.4, 100.9)
- moved U3 78.0 mm to (164.3, 100.5)
- moved C1 78.0 mm to (159.8, 104.9)
- moved R4 78.0 mm to (159.5, 100.2)
- moved JP1 74.2 mm to (145.6, 99.2), turned to -90 degrees
- moved R_{strain}2 65.5 mm to (170.1, 102.3)
- moved R_{strain}1 64.8 mm to (170.1, 112.0)
- moved H2 64.7 mm to (174.0, 118.5)
- moved H6 64.1 mm to (133.0, 118.5)
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Routing:
- net +5V: track 59.4 -> 77.2 mm
- net /CS1: track 12.3 -> 29.0 mm
- net /MISO: track 12.8 -> 23.8 mm, vias 0 -> 2
- net /V_{meas}+: track 11.7 -> 17.9 mm
- net /UDPI: track 10.1 -> 14.8 mm, vias 0 -> 2
- net /CS2: track 0.00 -> 3.38 mm, vias 0 -> 2
- net /MOSI: track 0.00 -> 3.38 mm, vias 0 -> 2
- net Net-(R_{G}1-Pad2): track 4.33 -> 6.75 mm
- net /V_{ref}: track 13.9 -> 14.7 mm
- net /SCK: track 16.6 -> 16.4 mm, vias 0 -> 2
- added copper zone on B.Cu, net GND
- added copper zone on F.Cu, net GND
Other:
- board size 52 x 68 mm -> 52 x 35.8 mm
- board text added: "LibreScale V0.1"
- board text added: "OLED"
